Commit message: updated wheel collisions and reduce slippage

File: openbase2_description/urdf/openbase2.xacro (robot description, xacro)
@@ -44,5 +44,5 @@
     <origin xyz="0.13 0.195 0.03" rpy="0 0 0"/>
     <geometry>
-      <mesh filename="file://$(find openbase2_description)/meshes/right_wheel.stl" scale="0.001 0.001 0.001"/>
+      <mesh filename="file://$(find openbase2_description)/meshes/right_wheel_collision.stl" scale="0.001 0.001 0.001"/>
     </geometry>
   </collision>
@@ -64,5 +64,5 @@
     <origin xyz="0.13 -0.195 0.03" rpy="0 0 0"/>
     <geometry>
-      <mesh filename="file://$(find openbase2_description)/meshes/left_wheel.stl" scale="0.001 0.001 0.001"/>
+      <mesh filename="file://$(find openbase2_description)/meshes/left_wheel_collision.stl" scale="0.001 0.001 0.001"/>
     </geometry>
   </collision>
